File: ADE9000_ESP32_DevKitC/ADE9000_ESP32_DevKitC.sch (EAGLE design)
At the start: 139 parts, among them IC1 24LC32A/SN, J9 ZX62-AB-5PA(31), Q1 MMBD4148SE, Q2 MMBD4148SE, Q3 MMBD4148SE, Q4 MMBD4148SE, Q5 MMBD4148SE, Q6 MMBD4148SE, Q7 MMBD4148SE, Q8 ECS-245.7-12-33Q-JES-TR, Q9 MMBD4148SE, U1 ADE9000ACPZ, U2 ADUM6404ARIZ, U3 SN74LV4T125PWR, U4 ADP122AUJZ-3.3-R7, U5 ADUM4151BRIZ, U6 SN74LV4T125PWR, U7 ESP32-WROOM-32, U8 ADP122AUJZ-3.3-R7

Commit message: esp+hive
Parts:
- removed C10, C14, C58: 0.1u, eagle-ltspice:CC0603
- removed C13, C57, C9: 10u, eagle-ltspice:C
- removed C26, C28: DNP, capacitors:C
- removed C31, C32: 0.022u, capacitors:C
- removed Q7, Q9: MMBD4148SE, DIODE_LED:DUAL_DIODE_SOT23-3
- removed R27, R28, R30, R52, R55, R56, R59: 10k, eagle-ltspice:RR0603
- removed SL4: 25.161.0253.0, GEEC_LibrariesCon_GEEC_Voltage:M02
- removed U8: ADP122AUJZ-3.3-R7, IC:ADP122AUJZ-3.3-R7
- added L2: 1500, inductors:FERRITE_BEAD0805
- J9: device Connectors:USB_MICRO -> connectors:USB_MICRO
- L1: device Inductors:FERRITE_BEAD0805 -> inductors:FERRITE_BEAD0805
- Q8: device Crystals:CRYSTAL_SMD128 -> crystals:CRYSTAL_SMD128
- R19, R20: value 5.1 -> 10k; device eagle-ltspice:R -> eagle-ltspice:RR0603
- R23, R24: value 0 -> 10k
- R25, R26: value 1k -> 10k
- U7: value ESP32-WROOM-32 -> ESP32-DEVKITC-32U; device ESP32-WROOM-32:ESP32-WROOM-32 -> ESP32-DEVKITC-32U:ESP32-DEVKITC-32U
Connections:
- removed net ESP3V3: R30.2
- removed net N$21: Q7.1, Q9.2, R19.1, R23.1, SL4.1
- removed net N$22: Q7.2, Q9.1, R20.2, R24.2, SL4.2
- removed net N$24: C28.2, R24.1, R26.1
- removed net N$25: C26.1, R23.2, R25.1
- removed net N$39: D2.C, S2.1
- removed net RESET_ARD: D1.C
- new net MODE_BUT: D2.A, R19.2, U7.IO34
- new net N$15: L2.1, SL5.2
- net GND: now also L2.2; no longer C26.2, C28.1, C31.2, C32.1, Q7.3, Q9.3, R19.2, R20.1, U8.GND, U8.NC
- net GNDA: now also S2.1, U7.GND1, U7.GND2, U7.GND3; no longer C10.2, C13.2, C14.2, C57.2, C58.2, C9.2, S2.2, U7.GND
- net INN: no longer C32.2, R26.2
- net INP: no longer C31.1, R25.2
- net IRQ0_ISO: now also R25.1; no longer R27.1
- net IRQ1_ISO: now also R26.1; no longer R28.1
- net N$10: now also D2.C, S2.2; no longer R30.1, U7.EN
- net RESET_ESP: now also D1.C; no longer R59.1
- net RESET_ISO: no longer D2.A
- net SCL_ARDUINO: now also R24.1; no longer R55.1
- net SDA_ARDUINO: now also R23.1; no longer R52.1
- net SS_ISO: now also R20.1; no longer R56.1
- net V+: now also R19.1, R20.2, R23.2, R24.2, R25.2, R26.2; no longer C13.1, C14.1, C57.1, C58.1, R27.2, R28.2, R52.2, R55.2, R56.2, R59.2, U8.VOUT
- net VCC: now also U7.EXT_5V; no longer C10.1, C9.1, U8.EN, U8.VIN
Other:
- moved on the sheet: D2, S2
