File: final module esp/ADE9000 Shield.brd (EAGLE design)
At the start: 105.4 x 66.2 mm, 128 parts, among them IC1 24LC32A/SN, J9 ZX62-AB-5PA(31), Q1 MMBD4148SE, Q2 MMBD4148SE, Q3 MMBD4148SE, Q4 MMBD4148SE, Q5 MMBD4148SE, Q6 MMBD4148SE, Q8 ECS-245.7-12-33Q-JES-TR, U1 ADE9000ACPZ, U2 ADUM6404ARIZ, U3 SN74LV4T125PWR, U4 ADP122AUJZ-3.3-R7, U5 ADUM4151BRIZ, U6 SN74LV4T125PWR, U7 ESP32-WROOM-32, U8 ADP122AUJZ-3.3-R7

Commit message: esp+hive
Parts:
- moved R27 24.1 mm to (96.8, 50.2)
- moved R52 19.2 mm to (97.9, 28.4)
- moved C1 16.3 mm to (106.9, 27.8), turned to 0 degrees
- moved R56 16.1 mm to (91.1, 28.2)
- moved R28 14.1 mm to (94.1, 50.9), turned to 90 degrees
- moved C7 12.4 mm to (104.8, 24.9), turned to 270 degrees
- moved R59 11.2 mm to (91.1, 50.0), turned to 180 degrees
- moved R69 10.1 mm to (86.0, 28.3)
- moved R55 9.55 mm to (103.8, 27.8), turned to 0 degrees
- moved C56 6.74 mm to (78.0, 42.8)
- moved C58 6.43 mm to (88.3, 50.5)
- moved R53 4.81 mm to (78.7, 40.1), turned to 180 degrees
- moved C62 2.77 mm to (102.7, 17.5), turned to 90 degrees
- moved C63 2.77 mm to (104.9, 17.8), turned to 90 degrees
- moved C57 2.08 mm to (86.0, 51.1)
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Routing:
- net V+: track 167.6 -> 204.2 mm, vias 5 -> 6
- net SDA_ARDUINO: track 37.9 -> 15.3 mm, vias 2 -> 0
- net RESET_ESP: track 19.0 -> 3.16 mm
- net MOSI_ISO: track 42.9 -> 30.0 mm, vias 6 -> 2
- net IRQ1_ISO: track 78.7 -> 67.3 mm
- net SS_ISO: track 37.5 -> 28.3 mm, vias 2 -> 0
- net VCC: track 87.4 -> 83.5 mm
- net SCLK_ISO: track 22.2 -> 24.1 mm
- net IRQ0_ISO: track 68.4 -> 69.7 mm
- net SCL_ARDUINO: track 24.5 -> 23.5 mm, vias 2 -> 0
